File: ESP32 Breakout/ESP32 Breakout.kicad_sch (KiCad schematic)
At the start: 5 parts, among them J1 Conn_01x05_Socket, J2 Conn_01x02_Socket, Q1 2N3904, U1 ESP32C3

Commit message: Update ESP32 Breakout.kicad_sch
Other:
- title: ESP32C3 Breakout Board -> ESP32 Breakout
Changed lines of the file:
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@@
 	(paper "A5")
 	(title_block
-		(title "ESP32C3 Breakout Board")
+		(title "ESP32 Breakout")
 		(date "2025-08-11")
 		(rev "1")

Commit message: Update to V1.1
Parts:
- added J3: Conn_01x05_Socket, Custom Footprints:JST_XH_B5B-XH-A_1x05_P2.50mm_Vertical, symbol Connector:Conn_01x05_Socket
Connections:
- net +5V: now also J3.1 (Pin_1)
- net GND: now also J3.2 (Pin_2), J3.5 (Pin_5)
- net SCL: now also J3.4 (Pin_4)
- net SDA: now also J3.3 (Pin_3)
Other:
- note added: "Display"
