File: PCBs/Expansion Board/AERIS Expansion Board.kicad_pcb (KiCad board)
At the start: 2 copper layers, 43 x 19 mm, 6 parts, among them J1 Conn_01x05_Socket, J2 Conn_01x05_Socket, J3 Conn_01x04_Pin, J4 Conn_01x04_Pin

Commit message: Update AERIS Expansion Board.kicad_pcb
Parts:
- moved REF** 1.21 mm to (123.0, 107.6)
- moved REF** 0.52 mm to (134.5, 107.3)
Other:
- board text added: "V1.0"
Changed lines of the file:
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@@
 			)
 		)
-		(model "/Users/alex/Downloads/BME280.step"
+		(model "/Users/alex/Documents/GitHub/AERIS/CAD/Reference/BME280.step"
 			(offset
 				(xyz 0 0 2.6)
@@
 			)
 		)
-		(model "/Users/alex/Downloads/SCD41.step"
+		(model "/Users/alex/Documents/GitHub/AERIS/CAD/Reference/SCD41.step"
 			(offset
 				(xyz 0 0 2.6)
@@
 	(footprint "Symbol:KiCad-Logo2_5mm_SilkScreen"
 		(layer "B.Cu")
-		(at 133.975796 107.334319 180)
+		(at 134.5 107.334319 180)
 		(descr "KiCad Logo")
 		(tags "Logo KiCad")
@@
 	(footprint "Symbol:OSHW-Logo2_7.3x6mm_SilkScreen"
 		(layer "B.Cu")
-		(at 121.813006 107.576766 180)
+		(at 123.024204 107.576766 180)
 		(descr "Open Source Hardware Symbol")
 		(tags "Logo Symbol OSHW")
@@
 		)
 	)
+	(gr_text "V1.0"
+		(at 118.524204 105 90)
+		(layer "B.SilkS")
+		(effects
+			(font
+				(size 1.5 1.5)
+				(thickness 0.2)
+				(bold yes)
+			)
+			(justify left bottom mirror)
+		)
+	)

Commit message: Update PCBs
Swap to just ESP32C6
Make footprint libraries project and not global
Parts:
- J1, J2: footprint Connector_JST:JST_XH_B5B-XH-A_1x05_P2.50mm_Vertical -> Library:JST_XH_B5B-XH-A_1x05_P2.50mm_Vertical
- J3, J4: footprint Connector_PinHeader_2.54mm:PinHeader_1x04_P2.54mm_Vertical -> Library:PinHeader_1x04_P2.54mm_Vertical
- REF**: footprint Symbol:KiCad-Logo2_5mm_SilkScreen -> Library:KiCad-Logo2_5mm_SilkScreen
- REF**: footprint Symbol:OSHW-Logo2_7.3x6mm_SilkScreen -> Library:OSHW-Logo2_7.3x6mm_SilkScreen
Changed lines of the file:
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@@
 	(net 3 "/SDA")
 	(net 4 "/SCL")
-	(footprint "Connector_PinHeader_2.54mm:PinHeader_1x04_P2.54mm_Vertical"
+	(footprint "Library:PinHeader_1x04_P2.54mm_Vertical"
 		(layer "F.Cu")
 		(at 132 117 90)
@@
 		)
 	)
-	(footprint "Connector_JST:JST_XH_B5B-XH-A_1x05_P2.50mm_Vertical"
+	(footprint "Library:JST_XH_B5B-XH-A_1x05_P2.50mm_Vertical"
 		(layer "F.Cu")
 		(at 113 105 -90)
@@
 		)
 	)
-	(footprint "Connector_PinHeader_2.54mm:PinHeader_1x04_P2.54mm_Vertical"
+	(footprint "Library:PinHeader_1x04_P2.54mm_Vertical"
 		(layer "F.Cu")
 		(at 119.5 117 90)
@@
 		)
 	)
-	(footprint "Connector_JST:JST_XH_B5B-XH-A_1x05_P2.50mm_Vertical"
+	(footprint "Library:JST_XH_B5B-XH-A_1x05_P2.50mm_Vertical"
 		(layer "F.Cu")
 		(at 105.5 105 -90)
@@
 		)
 	)
-	(footprint "Symbol:KiCad-Logo2_5mm_SilkScreen"
+	(footprint "Library:KiCad-Logo2_5mm_SilkScreen"
 		(layer "B.Cu")
 		(at 134.5 107.334319 180)
@@
 		(embedded_fonts no)
 	)
-	(footprint "Symbol:OSHW-Logo2_7.3x6mm_SilkScreen"
+	(footprint "Library:OSHW-Logo2_7.3x6mm_SilkScreen"
 		(layer "B.Cu")
 		(at 123.024204 107.576766 180)
